File: PCBs/Ai1_CC1000/Ai1_CC1000.kicad_sch (KiCad schematic)
At the start: 17 parts, among them J1 MCU_Cons, J2 MCU_D, J3 MCU_A, U1 CC1000, Y1 Crystal

Commit message: Switching1
Falta os switches das bobinas
Parts:
- removed AE1: Antenna, symbol Device:Antenna
- added C1_0, C1_3: 100nF, Capacitor_SMD:C_0603_1608Metric, symbol Device:C
- added C1_1, C1_4: 10nF, Capacitor_SMD:C_0603_1608Metric, symbol Device:C
- added C1_2, C1_5: 1nF, Capacitor_SMD:C_0603_1608Metric, symbol Device:C
- added C31_1: 15pF, Capacitor_SMD:C_0603_1608Metric, symbol Device:C
- added C31_2: 10pF, Capacitor_SMD:C_0603_1608Metric, symbol Device:C
- added C41_1: 8.2pF, Capacitor_SMD:C_0603_1608Metric, symbol Device:C
- added C42_1: 5.6pF, Capacitor_SMD:C_0603_1608Metric, symbol Device:C
- added C42_2: 4.7pF, Capacitor_SMD:C_0603_1608Metric, symbol Device:C
- added J4: RF_Control, symbol Connector_Generic:Conn_01x06
- added JP1: GND, symbol Jumper:Jumper_2_Open
- added JP2: VCC, symbol Jumper:Jumper_2_Open
- added L101_1: 33nH, Capacitor_SMD:C_0805_2012Metric, symbol Device:L
- added L101_2: 4.7nH, Capacitor_SMD:C_0805_2012Metric, symbol Device:L
- added L32_1: 68nH, Capacitor_SMD:C_0805_2012Metric, symbol Device:L
- added L32_2: 120nH, Capacitor_SMD:C_0805_2012Metric, symbol Device:L
- added L41_1: 6.2nH, Capacitor_SMD:C_0805_2012Metric, symbol Device:L
- added L41_2: 2.5nH, Capacitor_SMD:C_0805_2012Metric, symbol Device:L
- added SO1: VDA, symbol Device:Battery_Cell
- added SO2: VDD, symbol Device:Battery_Cell
- added U2, U3, U4, U5, U6, U8: ADG918BRM, Package_SO:MSOP-8_3x3mm_P0.65mm, symbol RF_Switch:ADG918BRM
- C171, C181: value C -> 18pF; footprint (none) -> Capacitor_SMD:C_0603_1608Metric
- C31_0: renamed from C31; value C -> 8.2pF; footprint (none) -> Capacitor_SMD:C_0603_1608Metric
- C41_0: renamed from C41; value C -> 2.2pF; footprint (none) -> Capacitor_SMD:C_0603_1608Metric
- C42_0: renamed from C42; value C -> 5.6pF; footprint (none) -> Capacitor_SMD:C_0603_1608Metric
- L101_0: renamed from L101; value L -> 56nH; footprint (none) -> Capacitor_SMD:C_0805_2012Metric
- L32_0: renamed from L32; value L -> 39nH; footprint (none) -> Capacitor_SMD:C_0805_2012Metric
- L41_0: renamed from L41; value L -> 20nH; footprint (none) -> Capacitor_SMD:C_0805_2012Metric
- Y1: value Crystal -> 14.7456MHz + 16pF Load
Connections:
- net GNDA: now also C1_0.1, C1_1.1, C1_2.1, JP1.2 (B), L32_1.2, L32_2.2, SO1.2 (-), U2.3 (GND), U2.6 (GND), U2.7 (GND), U3.3 (GND), U3.6 (GND), U3.7 (GND), U4.3 (GND), U4.6 (GND), U4.7 (GND), U5.3 (GND), U5.6 (GND), U5.7 (GND), U6.3 (GND), U6.6 (GND), U6.7 (GND), U8.3 (GND), U8.6 (GND), U8.7 (GND)
- net GNDD: now also C1_3.1, C1_4.1, C1_5.1, JP1.1 (A), SO2.2 (-)
- net IN_Matching: now also U2.4 (RFC); no longer C31_0.1, L32_0.1
- net OUT_Matching: now also U5.4 (RFC); no longer C41_0.2, C42_0.1, L41_0.1
- net VDD: now also C1_3.2, C1_4.2, C1_5.2, JP2.1 (A), SO2.1 (+)
- net VDDA: now also C1_0.2, C1_1.2, C1_2.2, C41_1.1, JP2.2 (B), L41_1.2, L41_2.2, SO1.1 (+), U2.1 (VDD), U3.1 (VDD), U4.1 (VDD), U5.1 (VDD), U6.1 (VDD), U8.1 (VDD)
- net 315MHz_In: now reaches C31_0.2
- net 315MHz_In: now also L32_0.1, U2.8 (RF1); no longer C42_0.2
- net L101_1: now reaches U1.10 (L1)
- net L101_1: no longer L101_0.1
- net L101_2: now reaches U1.11 (L2)
- net L101_2: no longer L101_0.2
- new net: U2.5 (RF2), U3.4 (RFC)
- new net: U4.4 (RFC), U5.5 (RF2)
- new net: U6.4 (RFC), U8.5 (RF2)
- new net 315Mhz_Out: C41_0.2, C42_0.2, L41_0.1, U5.8 (RF1)
- new net 433MHz_In: C31_1.2, L32_1.1, U3.8 (RF1)
- new net 433Mhz_Out: C41_1.2, C42_1.2, L41_1.1, U4.8 (RF1)
- new net 915MHz_In: C31_2.2, L32_2.1, U3.5 (RF2)
- new net 915Mhz_Out: C42_2.2, L41_2.1, U4.5 (RF2)
- new net C_RFS_1: J4.1 (Pin_1), U2.2 (CTRL)
- new net C_RFS_2: J4.2 (Pin_2), U3.2 (CTRL)
- new net C_RFS_3: J4.3 (Pin_3), U5.2 (CTRL)
- new net C_RFS_4: J4.4 (Pin_4), U4.2 (CTRL)
- new net C_RFS_5: J4.5 (Pin_5), U8.2 (CTRL)
- new net C_RFS_6: J4.6 (Pin_6), U6.2 (CTRL)
- new net L_315_1: L101_0.1
- new net L_315_2: L101_0.2
- new net L_433_1: L101_1.1
- new net L_433_2: L101_1.2
- new net L_915_1: L101_2.1
- new net L_915_2: L101_2.2
- new net To_Ant: U8.4 (RFC)
- new net To_Ant_315Mhz: C31_0.1, C42_0.1, U8.8 (RF1)
- new net To_Ant_433Mhz: C31_1.1, C42_1.1, U6.8 (RF1)
- new net To_Ant_915Mhz: C31_2.1, C42_2.1, U6.5 (RF2)
Other:
- note added: "315Mhz"
- note added: "433MHz"
- note added: "868-915MHz"
- note added: "Main IC"
- note added: "Matching TSSOP"
- note added: "Switching"
- note removed: "Lumped Matching"
- moved on the sheet: C171, C181, C281, C31_0, C41_0, C42_0, J1, J2, J3, L101_0, L32_0, L41_0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

Commit message: Com L switchs
Parts:
- removed J4: RF_Control, symbol Connector_Generic:Conn_01x06
- added J4: RF_Control, symbol Connector_Generic:Conn_01x08
- added U7, U9: ADG918BRM, Package_SO:MSOP-8_3x3mm_P0.65mm, symbol RF_Switch:ADG918BRM
Connections:
- net L_315_2 is gone; now on net L101_2: L101_0.2
- net L_433_2 is gone; now on net L101_2: L101_1.2
- net L_915_2 is gone; now on net L101_2: L101_2.2
- net C_RFS_1: now also J4.1 (Pin_1)
- net C_RFS_2: now also J4.2 (Pin_2)
- net C_RFS_3: now also J4.3 (Pin_3)
- net C_RFS_4: now also J4.4 (Pin_4)
- net C_RFS_5: now also J4.5 (Pin_5)
- net C_RFS_6: now also J4.6 (Pin_6)
- net GNDA: now also U7.3 (GND), U7.6 (GND), U7.7 (GND), U9.3 (GND), U9.6 (GND), U9.7 (GND)
- net L101_1: now also U9.4 (RFC)
- net L_315_1: now also U9.8 (RF1)
- net L_433_1: now also U7.8 (RF1)
- net L_915_1: now also U7.5 (RF2)
- net VDDA: now also U7.1 (VDD), U9.1 (VDD)
- new net: U7.4 (RFC), U9.5 (RF2)
- new net C_RFS_7: J4.7 (Pin_7), U9.2 (CTRL)
- new net C_RFS_8: J4.8 (Pin_8), U7.2 (CTRL)

Commit message: DRC LIMPO E SWITCH L101
Parts:
- removed J4: RF_Control, symbol Connector_Generic:Conn_01x08
- added J4: RF_Control, symbol Connector_Generic:Conn_01x10
- added J5: Ant_Con, symbol Connector_Generic:Conn_01x01
- added U10, U11: ADG918BRM, Package_SO:MSOP-8_3x3mm_P0.65mm, symbol RF_Switch:ADG918BRM
Connections:
- net C_RFS_1: now also J4.1 (Pin_1)
- net C_RFS_2: now also J4.2 (Pin_2)
- net C_RFS_3: now also J4.3 (Pin_3)
- net C_RFS_4: now also J4.4 (Pin_4)
- net C_RFS_5: now also J4.5 (Pin_5)
- net C_RFS_6: now also J4.6 (Pin_6)
- net C_RFS_7: now also J4.7 (Pin_7)
- net C_RFS_8: now also J4.8 (Pin_8)
- net GNDA: now also U10.3 (GND), U10.6 (GND), U10.7 (GND), U11.3 (GND), U11.6 (GND), U11.7 (GND)
- net L101_2: now also U11.4 (RFC); no longer L101_0.2, L101_1.2, L101_2.2
- net To_Ant: now also J5.1 (Pin_1)
- net VDDA: now also U10.1 (VDD), U11.1 (VDD)
- new net: U10.4 (RFC), U11.5 (RF2)
- new net C_RFS_10: J4.10 (Pin_10), U10.2 (CTRL)
- new net C_RFS_9: J4.9 (Pin_9), U11.2 (CTRL)
- new net L_315_2: L101_0.2, U11.8 (RF1)
- new net L_433_2: L101_1.2, U10.8 (RF1)
- new net L_915_2: L101_2.2, U10.5 (RF2)
Other:
- moved on the sheet: C171, C181, C1_0, C1_1, C1_2, C1_3, C1_4, C1_5, JP1, JP2, SO1, SO2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

Commit message: Crystal Escolhido
Parts:
- C281: footprint (none) -> Capacitor_SMD:C_0603_1608Metric
- J1: footprint (none) -> Connector_PinSocket_2.54mm:PinSocket_1x05_P2.54mm_Vertical
- J2, J3: footprint (none) -> Connector_PinSocket_2.54mm:PinSocket_1x01_P2.54mm_Vertical
- J4: footprint (none) -> Connector_PinSocket_2.54mm:PinSocket_2x05_P2.54mm_Vertical
- J5: footprint (none) -> Connector_Coaxial:SMA_Molex_73251-1153_EdgeMount_Horizontal
- JP1, JP2: footprint (none) -> Jumper:SolderJumper-2_P1.3mm_Open_TrianglePad1.0x1.5mm
- R131, R281: footprint (none) -> Resistor_SMD:R_0603_1608Metric
- SO1, SO2: footprint (none) -> TerminalBlock:TerminalBlock_MaiXu_MX126-5.0-02P_1x02_P5.00mm
- Y1: footprint (none) -> Crystal:Crystal_SMD_HC49-SD_HandSoldering

Commit message: innit layout
Parts:
- removed J5: Ant_Con, Connector_Coaxial:SMA_Molex_73251-1153_EdgeMount_Horizontal, symbol Connector_Generic:Conn_01x01
- added AE1: Antenna_Shield, Connector_Coaxial:SMA_Molex_73251-1153_EdgeMount_Horizontal, symbol Device:Antenna_Shield
- SO1, SO2: footprint TerminalBlock:TerminalBlock_MaiXu_MX126-5.0-02P_1x02_P5.00mm -> TerminalBlock_Phoenix:TerminalBlock_Phoenix_MPT-0,5-2-2.54_1x02_P2.54mm_Horizontal
Connections:
- net GNDA: now also AE1.2 (Shield)
- net To_Ant: now also AE1.1 (A)
Other:
- note added: "Having an RF Switch doesnt make much sense, seria melhor so ter antenas individuais"
Changed lines of the file:
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@@
 	(paper "A3")
 	(rectangle
+		(start 290.83 72.39)
+		(end 400.05 133.35)
+		(stroke
+			(width 0.254)
+			(type default)
+			(color 255 0 26 1)
+		)
+		(fill
+			(type none)
+		)
+	)
+	(rectangle
 		(start 236.22 24.13)
 		(end 283.21 60.96)
@@
 		)
 	)
+	(text "Having an RF Switch doesnt make much sense,\nseria melhor so ter antenas individuais\n"
+		(exclude_from_sim no)
+		(at 315.214 75.692 0)
+		(effects
+			(font
+				(size 1.27 1.27)
+			)
+		)
+	)
 	(text "315Mhz"
 		(exclude_from_sim no)
@@
 	(wire
 		(pts
+			(xy 232.41 241.3) (xy 234.95 241.3)
+		)
+		(stroke
+			(width 0)
+			(type default)
+		)
+	)
+	(wire
+		(pts
 			(xy 294.64 34.29) (xy 308.61 34.29)
 		)
@@
 	)
 	(label "To_Ant"
-		(at 240.03 236.22 0)
+		(at 232.41 241.3 180)
 		(effects
 			(font
 				(size 1.27 1.27)
 			)
-			(justify left bottom)
+			(justify right bottom)
 		)
 	)
@@
 	)
 	(symbol
-		(lib_id "Connector_Generic:Conn_01x01")
-		(at 234.95 236.22 180)
-		(unit 1)
-		(body_style 1)
-		(exclude_from_sim no)
-		(in_bom yes)
-		(on_board yes)
-		(in_pos_files yes)
-		(dnp no)
-		(fields_autoplaced yes)
-		(property "Reference" "J5"
-			(at 234.95 229.87 0)
-			(show_name no)
-			(do_not_autoplace no)
-			(effects
-				(font
-					(size 1.27 1.27)
-				)
-			)
-		)
-		(property "Value" "Ant_Con"
-			(at 234.95 232.41 0)
-			(show_name no)
-			(do_not_autoplace no)
-			(effects
-				(font
-					(size 1.27 1.27)
-				)
-			)
-		)
-		(property "Footprint" "Connector_Coaxial:SMA_Molex_73251-1153_EdgeMount_Horizontal"
-			(at 234.95 236.22 0)
-			(hide yes)
-			(show_name no)
-			(do_not_autoplace no)
-			(effects
-				(font
-					(size 1.27 1.27)
-				)
-			)
-		)
-		(property "Datasheet" ""
-			(at 234.95 236.22 0)
-			(hide yes)
-			(show_name no)
-			(do_not_autoplace no)
-			(effects
-				(font
-					(size 1.27 1.27)
-				)
-			)
-		)
-		(property "Description" "Generic connector, single row, 01x01, script generated (kicad-library-utils/schlib/autogen/connector/)"
-			(at 234.95 236.22 0)
-			(hide yes)
-			(show_name no)
-			(do_not_autoplace no)
-			(effects
-				(font
-					(size 1.27 1.27)
-				)
-			)
-		)
-		(pin "1"
-		)
-		(instances
-			(project "Ai1_CC1000"
-				(path "/076dc5cd-406b-4946-8ecf-b008a690dad8"
-					(reference "J5")
-					(unit 1)
-				)
-			)
-		)
-	)
-	(symbol
 		(lib_id "power:GNDA")
 		(at 242.57 181.61 0)
@@
 	)
 	(symbol
+		(lib_id "Device:Antenna_Shield")
+		(at 234.95 236.22 0)
+		(unit 1)
+		(body_style 1)
+		(exclude_from_sim no)
+		(in_bom yes)
+		(on_board yes)
+		(in_pos_files yes)
+		(dnp no)
+		(fields_autoplaced yes)
+		(property "Reference" "AE1"
+			(at 238.76 234.3149 0)
+			(show_name no)
+			(do_not_autoplace no)
+			(effects
+				(font
+					(size 1.27 1.27)
+				)
+				(justify left)
+			)
+		)
+		(property "Value" "Antenna_Shield"
+			(at 238.76 236.8549 0)
+			(show_name no)
+			(do_not_autoplace no)
+			(effects
+				(font
+					(size 1.27 1.27)
+				)
+				(justify left)
+			)
+		)
+		(property "Footprint" "Connector_Coaxial:SMA_Molex_73251-1153_EdgeMount_Horizontal"
+			(at 234.95 233.68 0)
+			(hide yes)
+			(show_name no)
+			(do_not_autoplace no)
+			(effects
+				(font
+					(size 1.27 1.27)
+				)
+			)
+		)
+		(property "Datasheet" ""
+			(at 234.95 233.68 0)
+			(hide yes)
+			(show_name no)
+			(do_not_autoplace no)
+			(effects
+				(font
+					(size 1.27 1.27)
+				)
+			)
+		)
+		(property "Description" "Antenna with extra pin for shielding"
+			(at 234.95 236.22 0)
+			(hide yes)
+			(show_name no)
+			(do_not_autoplace no)
+			(effects
+				(font
+					(size 1.27 1.27)
+				)
+			)
+		)
+		(pin "1"
+		)
+		(pin "2"
+		)
+		(instances
+			(project "Ai1_CC1000"
+				(path "/076dc5cd-406b-4946-8ecf-b008a690dad8"
+					(reference "AE1")
+					(unit 1)
+				)
+			)
+		)
+	)
+	(symbol
 		(lib_id "Device:L")
 		(at 133.35 248.92 0)
@@
 	)
 	(symbol
+		(lib_id "power:GNDA")
+		(at 237.49 241.3 0)
+		(unit 1)
+		(body_style 1)
+		(exclude_from_sim no)
+		(in_bom yes)
+		(on_board yes)
+		(in_pos_files yes)
+		(dnp no)
+		(property "Reference" "#PWR028"
+			(at 237.49 247.65 0)
+			(hide yes)
+			(show_name no)
+			(do_not_autoplace no)
+			(effects
+				(font
+					(size 1.27 1.27)
+				)
+			)
+		)
+		(property "Value" "GNDA"
+			(at 237.49 245.11 0)
+			(show_name no)
+			(do_not_autoplace no)
+			(effects
+				(font
+					(size 1.27 1.27)
+				)
+			)
+		)
+		(property "Footprint" ""
+			(at 237.49 241.3 0)
+			(hide yes)
+			(show_name no)
+			(do_not_autoplace no)
+			(effects
+				(font
+					(size 1.27 1.27)
+				)
+			)
+		)
+		(property "Datasheet" ""
+			(at 237.49 241.3 0)
+			(hide yes)
+			(show_name no)
+			(do_not_autoplace no)
+			(effects
+				(font
+					(size 1.27 1.27)
+				)
+			)
+		)
+		(property "Description" "Power symbol creates a global label with name \"GNDA\" , analog ground"
+			(at 237.49 241.3 0)
+			(hide yes)
+			(show_name no)
+			(do_not_autoplace no)
+			(effects
+				(font
+					(size 1.27 1.27)
+				)
+			)
+		)
+		(pin "1"
+		)
+		(instances
+			(project "Ai1_CC1000"
+				(path "/076dc5cd-406b-4946-8ecf-b008a690dad8"
+					(reference "#PWR028")
+					(unit 1)
+				)
+			)
+		)
+	)
+	(symbol
 		(lib_id "Device:C")
 		(at 120.65 245.11 90)
@@
 			)
 		)
-		(property "Footprint" "TerminalBlock:TerminalBlock_MaiXu_MX126-5.0-02P_1x02_P5.00mm"
+		(property "Footprint" "TerminalBlock_Phoenix:TerminalBlock_Phoenix_MPT-0,5-2-2.54_1x02_P2.54mm_Horizontal"
 			(at 340.36 41.656 90)
 			(hide yes)
@@
 			)
 		)
-		(property "Footprint" "TerminalBlock:TerminalBlock_MaiXu_MX126-5.0-02P_1x02_P5.00mm"
+		(property "Footprint" "TerminalBlock_Phoenix:TerminalBlock_Phoenix_MPT-0,5-2-2.54_1x02_P2.54mm_Horizontal"
 			(at 330.2 41.656 90)
 			(hide yes)
