File: PCBs/Ai1_CC1000/Ai1_CC1000.kicad_sch (KiCad schematic)
At the start: 49 parts, among them J1 MCU_Cons, J2 MCU_D, J3 MCU_A, J4 RF_Control, U1 CC1000, U10 ADG918BRM, U11 ADG918BRM, U2 ADG918BRM, U3 ADG918BRM, U4 ADG918BRM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

Commit message: Layout V2
Parts:
- removed U10, U11, U2, U3, U4, U5, U6, U7, U8, U9: ADG918BRM, Package_SO:MSOP-8_3x3mm_P0.65mm, symbol RF_Switch:ADG918BRM
- added IC1, IC10, IC2, IC3, IC4, IC5, IC6, IC7, IC8, IC9: BGS12WN6E6329XTSA1, Package_LGA:Infineon_PG-TSNP-6-10_0.7x1.1mm_0.7x1.1mm_P0.4mm, symbol BGS12WN6E6329XTSA1:BGS12WN6E6329XTSA1
Connections:
- net 315MHz_In: now also IC2.1 (RF2)
- net 315Mhz_Out: now also IC4.1 (RF2)
- net 433MHz_In: now also IC1.1 (RF2)
- net 433Mhz_Out: now also IC3.1 (RF2)
- net 915MHz_In: now also IC1.3 (RF1)
- net 915Mhz_Out: now also IC3.3 (RF1)
- net C_RFS_1: now also IC2.6 (CTRL)
- net C_RFS_10: now also IC9.6 (CTRL)
- net C_RFS_2: now also IC1.6 (CTRL)
- net C_RFS_3: now also IC4.6 (CTRL)
- net C_RFS_4: now also IC3.6 (CTRL)
- net C_RFS_5: now also IC6.6 (CTRL)
- net C_RFS_6: now also IC5.6 (CTRL)
- net C_RFS_7: now also IC8.6 (CTRL)
- net C_RFS_8: now also IC7.6 (CTRL)
- net C_RFS_9: now also IC10.6 (CTRL)
- net GNDA: now also IC1.2 (GND), IC10.2 (GND), IC2.2 (GND), IC3.2 (GND), IC4.2 (GND), IC5.2 (GND), IC6.2 (GND), IC7.2 (GND), IC8.2 (GND), IC9.2 (GND)
- net IN_Matching: now also IC2.5 (RFIN)
- net L101_1: now also IC8.5 (RFIN)
- net L101_2: now also IC10.5 (RFIN)
- net L_315_1: now also IC8.1 (RF2)
- net L_315_2: now also IC10.1 (RF2)
- net L_433_1: now also IC7.1 (RF2)
- net L_433_2: now also IC9.1 (RF2)
- net L_915_1: now also IC7.3 (RF1)
- net L_915_2: now also IC9.3 (RF1)
- net OUT_Matching: now also IC4.5 (RFIN)
- net To_Ant: now also IC6.5 (RFIN)
- net To_Ant_315Mhz: now also IC6.1 (RF2)
- net To_Ant_433Mhz: now also IC5.1 (RF2)
- net To_Ant_915Mhz: now also IC5.3 (RF1)
- net VDDA: now also IC1.4 (VDD), IC10.4 (VDD), IC2.4 (VDD), IC3.4 (VDD), IC4.4 (VDD), IC5.4 (VDD), IC6.4 (VDD), IC7.4 (VDD), IC8.4 (VDD), IC9.4 (VDD)
- new net: IC5.5 (RFIN), IC6.3 (RF1)
- new net: IC3.5 (RFIN), IC4.3 (RF1)
- new net: IC10.3 (RF1), IC9.5 (RFIN)
- new net: IC1.5 (RFIN), IC2.3 (RF1)
- new net: IC7.5 (RFIN), IC8.3 (RF1)
Other:
- moved on the sheet: AE1

Commit message: Layout V3 Antena needs attention
To check with prof
Antenas? Multiple?
Parts:
- removed J4: RF_Control, Connector_PinSocket_2.54mm:PinSocket_2x05_P2.54mm_Vertical, symbol Connector_Generic:Conn_01x10
- added J10, J11, J12, J13, J4, J5, J6, J7, J8, J9: RF_S_C, Connector_PinSocket_2.54mm:PinSocket_1x01_P2.54mm_Vertical, symbol Connector_Generic:Conn_01x01
Connections:
- net 315Mhz_Out: now also IC4.3 (RF1); no longer IC4.1 (RF2)
- net C_RFS_1: now also J4.1 (Pin_1)
- net C_RFS_10: now also J13.1 (Pin_1)
- net C_RFS_2: now also J5.1 (Pin_1)
- net C_RFS_3: now also J6.1 (Pin_1)
- net C_RFS_4: now also J7.1 (Pin_1)
- net C_RFS_5: now also J8.1 (Pin_1)
- net C_RFS_6: now also J9.1 (Pin_1)
- net C_RFS_7: now also J10.1 (Pin_1)
- net C_RFS_8: now also J11.1 (Pin_1)
- net C_RFS_9: now also J12.1 (Pin_1)
- net L_315_1: now also IC8.3 (RF1); no longer IC8.1 (RF2)
- net L_433_2: now also IC9.3 (RF1); no longer IC9.1 (RF2)
- net L_915_2: now also IC9.1 (RF2); no longer IC9.3 (RF1)
- net at IC3.5 (RFIN): now also IC4.1 (RF2); no longer IC4.3 (RF1)
- net DCLK: now reaches U1.24 (DCLK)
- net DCLK: now also J1.4 (Pin_4); no longer J1.1 (Pin_1)
- net DIO: now reaches U1.23 (DIO)
- net DIO: now also J1.5 (Pin_5); no longer J1.2 (Pin_2)
- net PALE: now reaches U1.27 (PALE)
- net PALE: now also J1.1 (Pin_1); no longer J1.3 (Pin_3)
- net PCLK: now reaches U1.25 (PCLK)
- net PCLK: now also J1.3 (Pin_3); no longer J1.4 (Pin_4)
- net PDATA: now reaches U1.26 (PDATA)
- net PDATA: now also J1.2 (Pin_2); no longer J1.5 (Pin_5)
- net at IC7.5 (RFIN): now also IC8.1 (RF2); no longer IC8.3 (RF1)
Other:
- moved on the sheet: J1

Commit message: PCB ready for fab 1 ?
Problemas atuais, antena e uma revisao sobre os traces, mas de acordo com a calculador de microstrip nenhum trace tem mais q 15EL ou seja menos de /4 entao nao devem desviar o matching
Connections:
- net To_Ant_433Mhz: now also IC5.3 (RF1); no longer IC5.1 (RF2)
- net To_Ant_915Mhz: now also IC5.1 (RF2); no longer IC5.3 (RF1)
Changed lines of the file:
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@@
+		)
+	)
+	(label "To_Ant_433Mhz"
+		(at 195.58 154.94 180)
+		(effects
+			(font
+				(size 1.27 1.27)
+			)
+			(justify right bottom)
 		)
 	)
@@
 		)
 	)
-	(label "To_Ant_433Mhz"
-		(at 195.58 149.86 180)
-		(effects
-			(font
-				(size 1.27 1.27)
-			)
-			(justify right bottom)
-		)
-	)
 	(label "L_315_2"
 		(at 160.02 166.37 0)
@@
 		)
 	)
-	(label "915MHz_In"
-		(at 198.12 113.03 180)
+	(label "To_Ant_915Mhz"
+		(at 195.58 149.86 180)
 		(effects
 			(font
@@
 		)
 	)
-	(label "To_Ant_915Mhz"
-		(at 195.58 154.94 180)
+	(label "915MHz_In"
+		(at 198.12 113.03 180)
 		(effects
 			(font
