File: PCBs/CC1101_Multx/CC1101_Multx.kicad_sch (KiCad schematic)
At the start: 45 parts, among them IC1 CC1101RGPR, IC2 ASWD-S2-0005-T, IC3 ASWD-S2-0005-T, IC4 ASWD-S2-0005-T, J1 MCU, J2 MCU, J3 MCU, J4 MCU, J5 MCU, J6 MCU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

Commit message: Layout V1
Parts:
- removed C126_2: 47pF, Capacitor_SMD:C_0402_1005Metric, symbol Device:C
- removed L125_2: 3.3nH, Inductor_SMD:L_0402_1005Metric, symbol Device:L
- added C4, C5: 27pF, Capacitor_SMD:C_0402_1005Metric, symbol Device:C
- L124_2: footprint Inductor_SMD:L_0402_1005Metric -> Inductor_SMD:L_0603_1608Metric
Connections:
- net 433_N: now also IC2.3 (RF1); no longer IC2.1 (RF2)
- net 868_N: now also IC2.1 (RF2); no longer IC2.3 (RF1)
- net AGND: now also C4.1, C5.1
- net at IC1.8 (XOSC_Q1), Y1.1: now also C4.2
- net at IC1.10 (XOSC_Q2), Y1.3: now also C5.2
