File: PCBs/CC1101_Multx/CC1101_Multx.kicad_sch (KiCad schematic)
At the start: 45 parts, among them IC1 CC1101RGPR, IC2 ASWD-S2-0005-T, IC3 ASWD-S2-0005-T, IC4 ASWD-S2-0005-T, J1 MCU, J2 MCU, J3 MCU, J4 MCU, J5 MCU, J6 MCU, J7 MCU, J8 MCU, J9 MCU, Y1 XRCGB26M000F1S2BR0

Commit message: BOM 1
Parts:
- AE1: footprint Connector_Coaxial:SMA_Molex_73251-1153_EdgeMount_Horizontal -> Connector_Coaxial:SMA_Molex_73251-2120_EdgeMount_Horizontal; LCSC Part # (none) -> C22467594
- BT1, J1, J2, J3, J4, J5, J6, J7, J8, J9: now not fitted; now left out of the parts list
- C1: LCSC Part # (none) -> C126521
- C121_1, C131_1: LCSC Part # (none) -> C88893
- C121_2: LCSC Part # (none) -> C710646
- C122_1: LCSC Part # (none) -> C2272083
- C122_2, C131_2: LCSC Part # (none) -> C710647
- C123_1: LCSC Part # (none) -> C161329
- C123_2: LCSC Part # (none) -> C76906
- C124_1, C125_1: LCSC Part # (none) -> C126503
- C124_2: LCSC Part # (none) -> C2941926
- C125_2: LCSC Part # (none) -> C76948
- C2: LCSC Part # (none) -> C2189775
- C3: LCSC Part # (none) -> C162190
- C4, C5: LCSC Part # (none) -> C710837
- C51: value 100n -> 100nF; LCSC Part # (none) -> C2189775
- IC1: LCSC Part # (none) -> C29953
- IC2, IC3, IC4: LCSC Part # (none) -> C47342120
- L121_1, L123_1, L131_1: LCSC Part # (none) -> C2043861
- L121_2, L123_2, L131_2: LCSC Part # (none) -> C2986278
- L122_1: LCSC Part # (none) -> C2044066
- L122_2, L132_2: LCSC Part # (none) -> C437365
- L124_2: LCSC Part # (none) -> C98068
- R171: LCSC Part # (none) -> C427251
- Y1: LCSC Part # (none) -> C7129840

Commit message: Layout new switch and BOM
Parts:
- IC2, IC3, IC4: footprint Library:ASWDS20005T -> Library:ASWS_S2_0002
Changed lines of the file:
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@@
 			)
 		)
-		(property "Footprint" "Library:ASWDS20005T"
+		(property "Footprint" "Library:ASWS_S2_0002"
 			(at 101.6 157.48 0)
 			(hide yes)
@@
 			)
 		)
-		(property "Footprint" "Library:ASWDS20005T"
+		(property "Footprint" "Library:ASWS_S2_0002"
 			(at 53.34 175.26 0)
 			(hide yes)
@@
 			)
 		)
-		(property "Footprint" "Library:ASWDS20005T"
+		(property "Footprint" "Library:ASWS_S2_0002"
 			(at 53.34 157.48 0)
 			(hide yes)

Commit message: V3 Fasivel
Parts:
- removed IC2, IC3, IC4: ASWD-S2-0005-T, Library:ASWS_S2_0002, symbol New_Library:ASWD-S2-0005-T
- added U1, U2, U3: 4259-63, Library:SC-70-6_PSM-M, symbol New_Library:4259-63
- AE1: footprint Connector_Coaxial:SMA_Molex_73251-2120_EdgeMount_Horizontal -> Library:SMA_CONSMA020_062_G
- BT1: footprint TerminalBlock_Phoenix:TerminalBlock_Phoenix_MPT-0,5-2-2.54_1x02_P2.54mm_Horizontal -> Connector_PinHeader_2.54mm:PinHeader_1x02_P2.54mm_Vertical
Connections:
- net 433_A: now also U2.1 (RF1)
- net 433_N: now also U1.3 (RF2)
- net 433_P: now also U3.1 (RF1)
- net 868_A: now also U2.3 (RF2)
- net 868_N: now also U1.1 (RF1)
- net 868_P: now also U3.3 (RF2)
- net AGND: now also U1.2 (GND), U2.2 (GND), U3.2 (GND)
- net AVDD: now also U1.6 (*CTRL/VDD), U2.6 (*CTRL/VDD), U3.6 (*CTRL/VDD)
- net RF_N: now also U1.5 (RFC)
- net RF_P: now also U3.5 (RFC)
- net To_Ant: now also U2.5 (RFC)
- net at J9.1 (Pin_1): now also U2.4 (CTRL)
- net at J8.1 (Pin_1): now also U3.4 (CTRL)
- net at J7.1 (Pin_1): now also U1.4 (CTRL)
Other:
- moved on the sheet: BT1, C1, C2, C3, J7, J8, J9

Commit message: pord please
Parts:
- AE1: Digikey Part # (none) -> 343-CONSMA020.062-G-ND; Part Name (none) -> CONSMA020.062-G
- C1: Digikey Part # (none) -> 490-GRM155C71A105KE11JCT-ND; Part Name (none) -> GRM155C71A105KE11J
- C121_1, C131_1: Digikey Part # (none) -> 490-11216-1-ND; Part Name (none) -> GJM1555C1H3R9WB01D
- C121_2: Digikey Part # (none) -> 490-GCM1555C1H1R0JA16DCT-ND; Part Name (none) -> GCM1555C1H1R0JA16D
- C122_1: Digikey Part # (none) -> 490-GCQ1555C1H8R2WB01DCT-ND; Part Name (none) -> GCQ1555C1H8R2WB01D
- C122_2, C131_2: Digikey Part # (none) -> 490-16452-1-ND; Part Name (none) -> GCM1555C1H1R5JA16D
- C123_1: Digikey Part # (none) -> 490-11225-1-ND; Part Name (none) -> GJM1555C1H5R6BB01D
- C123_2: Digikey Part # (none) -> 490-8097-1-ND; Part Name (none) -> GJM1555C1H3R3BB01D
- C124_1, C125_1: Digikey Part # (none) -> 490-4927-1-ND; Part Name (none) -> GCM1555C1H221JA16D
- C124_2: Digikey Part # (none) -> 490-14349-1-ND; Part Name (none) -> GCM1555C1H101FA16D
- C125_2: Digikey Part # (none) -> 490-5924-1-ND; Part Name (none) -> GRM1555C1H120JA01D
- C2, C51: Digikey Part # (none) -> 490-GRM155C71H104JE19DCT-ND; Part Name (none) -> GRM155C71H104JE19D
- C3: Digikey Part # (none) -> 490-7763-1-ND; Part Name (none) -> GRM155R71H103JA88D
- C4, C5: Digikey Part # (none) -> 490-6176-1-ND; Part Name (none) -> GRM1555C1E270JA01D
- IC1: Digikey Part # (none) -> 296-35718-1-ND; Part Name (none) -> CC1101RGPR
- L121_1, L123_1, L131_1: Digikey Part # (none) -> 490-15374-1-ND; Part Name (none) -> LQW15AN27NJ8ZD
- L121_2, L123_2, L131_2: Digikey Part # (none) -> 490-LQW15AN12NJ80DCT-ND; Part Name (none) -> LQW15AN12NJ80D
- L122_1: Digikey Part # (none) -> 490-15363-1-ND; Part Name (none) -> LQW15AN22NG8ZD
- L122_2, L132_2: Part Name (none) -> LQW15CN18NJ00D
- L124_2: Digikey Part # (none) -> 490-6861-1-ND; Part Name (none) -> LQW18AN12NG00D
- R171: Digikey Part # (none) -> P124494CT-ND; Part Name (none) -> ERJ-PA2F5602X
- Y1: Digikey Part # (none) -> 490-XRCGB26M000F1S2BR0CT-ND; Part Name (none) -> XRCGB26M000F1S2BR0

Commit message: tweaks
Parts:
- L122_2, L132_2: Digikey Part # (none) -> 490-15348-1-ND; Part Name LQW15CN18NJ00D -> LQW15AN18NJ8ZD
Changed lines of the file:
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@@
 			)
 		)
-		(property "Digikey Part #" ""
+		(property "Digikey Part #" "490-15348-1-ND"
 			(at 149.86 97.79 90)
 			(hide yes)
@@
 			)
 		)
-		(property "Part Name" "LQW15CN18NJ00D"
+		(property "Part Name" "LQW15AN18NJ8ZD"
 			(at 149.86 97.79 90)
 			(hide yes)
@@
 			)
 		)
-		(property "Digikey Part #" ""
-			(at 139.7 114.3 0)
-			(hide yes)
-			(show_name no)
-			(do_not_autoplace no)
-			(effects
-				(font
-					(size 1.27 1.27)
-				)
-			)
-		)
-		(property "Part Name" "LQW15CN18NJ00D"
-			(at 139.7 114.3 0)
-			(hide yes)
+		(property "Digikey Part #" "490-15348-1-ND"
+			(at 139.7 114.3 0)
+			(hide yes)
+			(show_name no)
+			(do_not_autoplace no)
+			(effects
+				(font
+					(size 1.27 1.27)
+				)
+			)
+		)
+		(property "Part Name" "LQW15AN18NJ8ZD"
+			(at 139.7 114.3 0)
+			(hide yes)

Commit message: ups switches
Parts:
- U1, U2, U3: Digikey Part # (none) -> 1046-1011-1-ND; Part Name (none) -> 4259-63
Changed lines of the file:
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@@
 			)
 		)
-		(property "Digikey Part #" ""
+		(property "Digikey Part #" "1046-1011-1-ND"
 			(at 24.13 158.75 0)
 			(hide yes)
@@
 			)
 		)
-		(property "Part Name" ""
+		(property "Part Name" "4259-63"
 			(at 24.13 158.75 0)
 			(hide yes)
@@
 			)
 		)
-		(property "Digikey Part #" ""
+		(property "Digikey Part #" "1046-1011-1-ND"
 			(at 64.77 181.61 0)
 			(hide yes)
@@
 			)
 		)
-		(property "Part Name" ""
+		(property "Part Name" "4259-63"
 			(at 64.77 181.61 0)
 			(hide yes)
@@
 			)
 		)
-		(property "Digikey Part #" ""
+		(property "Digikey Part #" "1046-1011-1-ND"
 			(at 96.52 158.75 0)
 			(hide yes)
@@
 			)
 		)
-		(property "Part Name" ""
+		(property "Part Name" "4259-63"
 			(at 96.52 158.75 0)
 			(hide yes)

Commit message: 2ants prod
Parts:
- removed J9: MCU, Connector_PinHeader_2.54mm:PinHeader_1x01_P2.54mm_Vertical, symbol Connector:Conn_01x01_Pin
- removed U2: 4259-63, Library:SC-70-6_PSM-M, symbol New_Library:4259-63
- added AE2: Antenna_Shield, Library:SMA_CONSMA020_062_G, symbol Device:Antenna_Shield
Connections:
- net To_Ant is gone; now on net 433_A: AE1.1 (A)
- net 868_A: now also AE2.1 (A)
- net AGND: now also AE2.2 (Shield)
Other:
- moved on the sheet: J8, U3
