File: PCBs/CC1101_Multx/CC1101_Multx.kicad_pcb (KiCad board)
At the start: 4 copper layers, 35.4 x 25.9 mm, 50 parts, among them IC1 CC1101RGPR, J1 MCU, J2 MCU, J3 MCU, J4 MCU, J5 MCU, J6 MCU, J7 MCU, J8 MCU, J9 MCU, U1 4259-63, U3 4259-63, Y1 XRCGB26M000F1S2BR0

Commit message: symetric
Parts:
- removed the REF** at (170.8, 71.4)
- removed the REF** at (170.8, 89.5)
- moved REF** 6.43 mm to (146.3, 69.5)
- moved REF** 6.18 mm to (146.3, 90.4)
- moved AE1 5.54 mm to (171.4, 70.2), turned to 90 degrees
- moved C125_1 2.31 mm to (171.4, 76.5)
- moved C5 1.78 mm to (158.6, 88.9), turned to 45 degrees
- moved C123_1 1.69 mm to (170.9, 78.0)
- moved C4 1.59 mm to (155.7, 88.7), turned to 135 degrees
- moved L131_1 1.09 mm to (168.1, 78.9)
- moved L123_1 1.08 mm to (171.4, 79.6)
- moved C122_1 0.91 mm to (171.9, 81.1), turned to 180 degrees
- moved Y1 0.44 mm to (157.1, 87.5), turned to -45 degrees
- moved C121_1 0.36 mm to (168.1, 85.5)
- moved L122_1 0.24 mm to (170.9, 82.2)
Routing:
- net Net-(J7-Pin_1): track 32.0 -> 19.1 mm
- net Net-(J8-Pin_1): track 26.3 -> 15.6 mm
- net /433_A: track 4.05 -> 5.95 mm
- net Net-(C121_1-Pad2): track 7.22 -> 8.83 mm
- net /AGND: track 24.8 -> 23.3 mm
- net Net-(IC1-XOSC_Q2): track 4.23 -> 5.46 mm
- net Net-(C123_1-Pad2): track 3.33 -> 2.09 mm
- net Net-(C122_1-Pad2): track 3.37 -> 2.13 mm
- net /AVDD: track 11.8 -> 12.4 mm
Other:
- board size 35.4 x 25.9 mm -> 35.4 x 26.1 mm

Commit message: latest PCB and noted
Routing:
- net /AGND: track 23.3 -> 24.1 mm, vias 144 -> 145
Changed lines of the file:
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@@
 		(start 143.56 66.82)
 		(end 179 92.89)
-		(radius 2.8)
+		(radius 2.5)
 		(stroke
 			(width 0.05)
@@
 	)
 	(segment
+		(start 156.596 79.9736)
+		(end 156.596 80.023604)
+		(width 0.2)
+		(layer "F.Cu")
+		(net "/AGND")
+	)
+	(segment
 		(start 151.5136 83.1596)
 		(end 151.5136 79.9592)
@@
 	)
 	(segment
-		(start 156.096 79.9736)
-		(end 156.096 81.3736)
+		(start 157.596 80.8736)
+		(end 157.596 79.9736)
 		(width 0.2)
 		(layer "F.Cu")
@@
 	)
 	(segment
-		(start 157.596 80.8736)
-		(end 156.596 81.8736)
+		(start 156.596 80.023604)
+		(end 155.671002 80.948602)
 		(width 0.2)
 		(layer "F.Cu")
@@
 	)
 	(segment
+		(start 155.671002 80.948602)
+		(end 156.596 81.8736)
+		(width 0.2)
+		(layer "F.Cu")
+		(net "/AGND")
+	)
+	(segment
 		(start 156.204449 89.186228)
 		(end 156.494928 89.476707)
@@
 	)
 	(segment
-		(start 163.710076 83.989957)
-		(end 163.950819 84.2307)
+		(start 156.096 81.3736)
+		(end 156.096 79.9736)
 		(width 0.2)
 		(layer "F.Cu")
@@
 	)
 	(segment
-		(start 157.596 79.9736)
-		(end 157.596 80.8736)
+		(start 163.710076 83.989957)
+		(end 163.950819 84.2307)
 		(width 0.2)
 		(layer "F.Cu")
@@
 	)
 	(segment
-		(start 156.596 79.9736)
-		(end 156.596 81.8736)
+		(start 156.596 81.8736)
+		(end 156.096 81.3736)
 		(width 0.2)
 		(layer "F.Cu")
@@
 	)
 	(segment
-		(start 156.096 81.3736)
-		(end 156.596 81.8736)
+		(start 157.14 86.666827)
+		(end 157.015973 86.5428)
 		(width 0.2)
 		(layer "F.Cu")
@@
 	)
 	(segment
-		(start 157.14 86.666827)
-		(end 157.015973 86.5428)
+		(start 157.5096 80.96)
+		(end 157.596 80.8736)
+		(width 0.2)
+		(layer "F.Cu")
+		(net "/AGND")
+	)
+	(segment
+		(start 157.5 80.96)
+		(end 157.5096 80.96)
 		(width 0.2)
 		(layer "F.Cu")
@@
 	)
 	(segment
+		(start 157.5 80.9696)
+		(end 156.596 81.8736)
+		(width 0.2)
+		(layer "F.Cu")
+		(net "/AGND")
+	)
+	(segment
 		(start 157.0736 77.6712)
 		(end 157.8336 77.6712)
@@
 	)
 	(segment
+		(start 157.5 80.96)
+		(end 157.5 80.9696)
+		(width 0.2)
+		(layer "F.Cu")
+		(net "/AGND")
+	)
+	(segment
 		(start 157.228105 89.50784)
 		(end 157.228105 88.381278)
@@
 	)
 	(via
-		(at 151.6 83.74)
+		(at 151.53 83.84)
 		(size 0.6)
 		(drill 0.3)
@@
 	)
 	(via
-		(at 154.08 83.72)
-		(size 0.6)
-		(drill 0.3)
-		(layers "F.Cu" "B.Cu")
-		(free yes)
-		(teardrops
-			(best_length_ratio 0.5)
-			(max_length 1)
-			(best_width_ratio 1)
-			(max_width 0.5)
-			(curved_edges yes)
-			(filter_ratio 0.9)
-			(enabled no)
-			(allow_two_segments yes)
-			(prefer_zone_connections yes)
-		)
-		(net "/AGND")
-	)
-	(via
 		(at 154.94 68.58)
 		(size 0.6)
@@
 	)
 	(via
+		(at 157.5 80.96)
+		(size 0.6)
+		(drill 0.3)
+		(layers "F.Cu" "B.Cu")
+		(net "/AGND")
+	)
+	(via
 		(at 167.64 73.66)
 		(size 0.6)
@@
 	)
 	(via
+		(at 155.671002 80.948602)
+		(size 0.6)
+		(drill 0.3)
+		(layers "F.Cu" "B.Cu")
+		(net "/AGND")
+	)
+	(via
 		(at 165.1 88.9)
 		(size 0.6)
@@
 	(segment
 		(start 161.25 82.65)
-		(end 161.24 82.66)
+		(end 161.06 82.46)
 		(width 0.2)
 		(layer "B.Cu")
@@
 	)
 	(segment
-		(start 154.12 82.66)
-		(end 150.49 86.29)
+		(start 156.844529 82.4736)
+		(end 156.347471 82.4736)
+		(width 0.2)
+		(layer "B.Cu")
+		(net "Net-(J8-Pin_1)")
+	)
+	(segment
+		(start 161.06 82.46)
+		(end 156.858129 82.46)
 		(width 0.2)
 		(layer "B.Cu")
@@
 	)
 	(segment
-		(start 161.24 82.66)
-		(end 154.12 82.66)
+		(start 156.347471 82.4736)
+		(end 156.333871 82.46)
+		(width 0.2)
+		(layer "B.Cu")
+		(net "Net-(J8-Pin_1)")
+	)
+	(segment
+		(start 154.32 82.46)
+		(end 150.49 86.29)
+		(width 0.2)
+		(layer "B.Cu")
+		(net "Net-(J8-Pin_1)")
+	)
+	(segment
+		(start 156.858129 82.46)
+		(end 156.844529 82.4736)
+		(width 0.2)
+		(layer "B.Cu")
+		(net "Net-(J8-Pin_1)")
+	)
+	(segment
+		(start 156.333871 82.46)
+		(end 154.32 82.46)
 		(width 0.2)
 		(layer "B.Cu")
@@
 	)
 	(zone
+		(layer "F.Cu")
+		(hatch edge 0.5)
+		(connect_pads yes
+			(clearance 0)
+		)
+		(min_thickness 0.25)
+		(keepout
+			(tracks allowed)
+			(vias allowed)
+			(pads allowed)
+			(copperpour not_allowed)
+			(footprints allowed)
+		)
+		(placement
+			(enabled no)
+			(sheetname "")
+		)
+		(fill
+			(thermal_gap 0.5)
+			(thermal_bridge_width 0.5)
+			(island_removal_mode 0)
+		)
+		(polygon
+			(pts
+				(xy 153.87 83.32) (xy 154.8 83.51) (xy 153.55 84.9) (xy 151.6 84.34) (xy 152.17 83.74)
+			)
+		)
+	)
+	(zone
