File: PCBs/BandPass_CSRF/BandPass_CSRF.kicad_sch (KiCad schematic)
At the start: 10 parts, among them J1 Conn_Coaxial, J2 Conn_Coaxial

Commit message: one and done
Parts:
- added J3, J4, J5, J6: Conn_Coaxial, Connector_Coaxial:SMA_Molex_73251-2120_EdgeMount_Horizontal, symbol Connector:Conn_Coaxial
- added Z10, Z12, Z14, Z16, Z18, Z20, Z22, Z24: L, Capacitor_SMD:C_0805_2012Metric_Pad1.18x1.45mm_HandSolder, symbol Device:R
- added Z11, Z13, Z15, Z17, Z19, Z21, Z23, Z9: C, Capacitor_SMD:C_0805_2012Metric_Pad1.18x1.45mm_HandSolder, symbol Device:R
- renumbered J2 to J1, J1 to J2
Connections:
- net GND renamed GND1
- new net: J3.1 (In), Z10.1, Z11.1, Z9.1
- new net: Z12.2, Z13.1, Z14.1, Z15.1
- new net: J5.1 (In), Z17.1, Z18.1, Z19.1
- new net: Z11.2, Z12.1
- new net: Z23.2, Z24.1
- new net: J6.1 (In), Z24.2
- new net: Z19.2, Z20.1
- new net: Z20.2, Z21.1, Z22.1, Z23.1
- new net: J4.1 (In), Z16.2
- new net: Z15.2, Z16.1
- new net GND2: J3.2 (Ext), J4.2 (Ext), Z10.2, Z13.2, Z14.2, Z9.2
- new net GND3: J5.2 (Ext), J6.2 (Ext), Z17.2, Z18.2, Z21.2, Z22.2
Other:
- note added: "Exemplo: https://markimicrowave.com/technical-resources/tools/lc-filter-design-tool/"
- moved on the sheet: J1, J2, Z1, Z2, Z3, Z4, Z5, Z6, Z7, Z8

Commit message: FinalPLS
Parts:
- J1, J2, J3, J4, J5, J6: footprint Connector_Coaxial:SMA_Molex_73251-2120_EdgeMount_Horizontal -> Library:SMA_CONSMA020_062_G
Other:
- note added: "https://www.digikey.pt/en/products/detail/te-connectivity-linx/CONSMA020-062-G/11482822"
